File: _autosave-principal_sm13.kicad_pcb (KiCad board)
At the start: 2 copper layers, 67 parts, among them J1 CN_ARM, J2 CN_POLE, P1 CONN_10X2, P2 SPI, Q1 BC807, Q2 BC807, Q3 BC807, Q4 BC807, U1 AD8397ARZ, U2 AD8397ARZ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

Commit message: cambios en el placement
Parts:
- P1, P2: moved to B.Cu
- moved P1 5.41 mm to (7.60, -63.0), turned to 270 degrees
- moved P2 4.46 mm to (-28.5, -63.0), turned to 270 degrees
- moved Q1 0.60 mm to (70.0, -91.4)
- moved Q2 0.60 mm to (70.0, -81.5)
- moved Q3 0.60 mm to (13.7, -91.5)
- moved Q4 0.60 mm to (13.7, -82.0)
