File: RDC_POLE.sch (KiCad schematic (older format))
At the start: 36 parts, among them J2 RESOLVER POLE, Q3 BC807, Q4 BC807, U2 AD8397ARZ, X2 8.192MHz

Commit message: cambiados capacitores electroliticos por tantalio (unpolarized). Agrandado footprint test pads, generado BOM, 35 vias
Parts:
- C14, C20, C25: symbol Device:CP1 -> Device:C
- C18: footprint Capacitor_SMD:CP_Elec_4x5.4 -> Capacitor_SMD:C_1206_3216Metric_Pad1.42x1.75mm_HandSolder; symbol Device:CP1 -> Device:C
- TP10, TP11, TP12, TP13, TP14, TP15: footprint TestPoint:TestPoint_THTPad_1.0x1.0mm_Drill0.5mm -> TestPoint:TestPoint_THTPad_1.5x1.5mm_Drill0.7mm
Connections:
- wire segments 125 -> 124
Changed lines of the file:
@@
 $EndComp
 $Comp
-L Device:CP1 C?
+L Device:C C?
 U 1 1 5EFA84B3
 P 4250 1800
@@
 Text Label 5050 2050 2    60   ~ 0
 AGND
-Connection ~ 4250 1650
-Wire Wire Line
-	4250 1650 4250 1750
 $Comp
 L Device:R R?
@@
 NoConn ~ 3150 3300
 $Comp
-L Device:CP1 C?
+L Device:C C?
 U 1 1 5F08F1CC
 P 3800 6500
@@
 $EndComp
 $Comp
-L Device:CP1 C?
+L Device:C C?
 U 1 1 5F08F1CD
 P 1700 4250
@@
 $EndComp
 $Comp
-L Device:CP1 C?
+L Device:C C?
 U 1 1 5EF54A0E
 P 1700 3600
@@
 F 0 "C18" H 1750 3700 50  0000 L CNN
 F 1 "10µ" H 1750 3500 50  0000 L CNN
-F 2 "Capacitor_SMD:CP_Elec_4x5.4" H 1700 3600 60  0000 C CNN
+F 2 "Capacitor_SMD:C_1206_3216Metric_Pad1.42x1.75mm_HandSolder" H 1700 3600 60  0000 C CNN
 F 3 "~" H 1700 3600 60  0000 C CNN
 	1    1700 3600
@@
 F 0 "TP14" V 9904 3138 50  0000 L CNN
 F 1 "TPEXCPOLE" V 9995 3138 50  0000 L CNN
-F 2 "TestPoint:TestPoint_THTPad_1.0x1.0mm_Drill0.5mm" H 10150 2950 50  0001 C CNN
+F 2 "TestPoint:TestPoint_THTPad_1.5x1.5mm_Drill0.7mm" H 10150 2950 50  0001 C CNN
 F 3 "~" H 10150 2950 50  0001 C CNN
 	1    9950 2950
@@
 F 0 "TP15" V 9904 5638 50  0000 L CNN
 F 1 "TPEXCLOPOLE" V 9995 5638 50  0000 L CNN
-F 2 "TestPoint:TestPoint_THTPad_1.0x1.0mm_Drill0.5mm" H 10150 5450 50  0001 C CNN
+F 2 "TestPoint:TestPoint_THTPad_1.5x1.5mm_Drill0.7mm" H 10150 5450 50  0001 C CNN
 F 3 "~" H 10150 5450 50  0001 C CNN
 	1    9950 5450
@@
 F 0 "TP10" V 3300 2600 50  0000 L CNN
 F 1 "TPCOSPOLE" V 3350 2900 50  0000 L CNN
-F 2 "TestPoint:TestPoint_THTPad_1.0x1.0mm_Drill0.5mm" H 3550 2700 50  0001 C CNN
+F 2 "TestPoint:TestPoint_THTPad_1.5x1.5mm_Drill0.7mm" H 3550 2700 50  0001 C CNN
 F 3 "~" H 3550 2700 50  0001 C CNN
 	1    3350 2700
@@
 F 0 "TP11" V 3400 2600 50  0000 L CNN
 F 1 "TPCOSLOPOLE" V 3450 2900 50  0000 L CNN
-F 2 "TestPoint:TestPoint_THTPad_1.0x1.0mm_Drill0.5mm" H 3650 2700 50  0001 C CNN
+F 2 "TestPoint:TestPoint_THTPad_1.5x1.5mm_Drill0.7mm" H 3650 2700 50  0001 C CNN
 F 3 "~" H 3650 2700 50  0001 C CNN
 	1    3450 2700
@@
 F 0 "TP12" V 3600 2600 50  0000 L CNN
 F 1 "TPSINLOPOLE" V 3650 2900 50  0000 L CNN
-F 2 "TestPoint:TestPoint_THTPad_1.0x1.0mm_Drill0.5mm" H 3850 2700 50  0001 C CNN
+F 2 "TestPoint:TestPoint_THTPad_1.5x1.5mm_Drill0.7mm" H 3850 2700 50  0001 C CNN
 F 3 "~" H 3850 2700 50  0001 C CNN
 	1    3650 2700
@@
 F 0 "TP13" V 3700 2600 50  0000 L CNN
 F 1 "TPSINPOLE" V 3750 2900 50  0000 L CNN
-F 2 "TestPoint:TestPoint_THTPad_1.0x1.0mm_Drill0.5mm" H 3950 2700 50  0001 C CNN
+F 2 "TestPoint:TestPoint_THTPad_1.5x1.5mm_Drill0.7mm" H 3950 2700 50  0001 C CNN
 F 3 "~" H 3950 2700 50  0001 C CNN
 	1    3750 2700
